File: hardware/moisture.kicad_pcb (KiCad board)
At the start: 2 copper layers, 15 x 85 mm, 31 parts, among them P1 CON-SENSOR2, P2 DEBUG, P3 BOOT, Q1 Oscillator, U1 XMC1XXX24, U2 MCP3425

Commit message: Add 3d information (fam)
Parts:
- U2: footprint SOT23-6 -> kicad-libraries:SOT23-6
Changed lines of the file:
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@@
-(kicad_pcb (version 4) (host pcbnew 4.0.6-e0-6349~53~ubuntu16.04.1)
+(kicad_pcb (version 4) (host pcbnew 4.0.2+dfsg1-stable)
   (general
     (links 71)
@@
     )
   )
-  (module kicad-libraries:SOT363 (layer F.Cu)
-    (at 136.7 91 270)
-    (attr smd)
-    (fp_text reference D2 (at 0.35 0 360) (layer F.Fab)
-      (effects (font (size 0.2 0.2) (thickness 0.05)))
-    )
-    (fp_text value BAT54TW (at 0.025 0.125 360) (layer F.Fab)
-      (effects (font (size 0.2 0.2) (thickness 0.05)))
-    )
-    (fp_circle (center -0.25 -0.7) (end -0.2 -0.65) (layer F.Fab) (width 0.05))
-    (fp_line (start -0.65 -1.1) (end 0.65 -1.1) (layer F.Fab) (width 0.05))
-    (fp_line (start 0.65 -1.1) (end 0.65 1.1) (layer F.Fab) (width 0.05))
-    (fp_line (start 0.65 1.1) (end -0.65 1.1) (layer F.Fab) (width 0.05))
-    (fp_line (start -0.65 1.1) (end -0.65 -1.1) (layer F.Fab) (width 0.05))
-    (pad 1 smd rect (at -0.9 -0.75 270) (size 0.6 0.6) (layers F.Cu F.Paste F.Mask)
-      (net 19 "Net-(D2-Pad1)"))
-    (pad 3 smd rect (at -0.9 0.75 270) (size 0.6 0.6) (layers F.Cu F.Paste F.Mask)
-      (net 25 SIG))
-    (pad 4 smd rect (at 0.9 0.75 270) (size 0.6 0.6) (layers F.Cu F.Paste F.Mask)
-      (net 17 "Net-(C10-Pad1)"))
-    (pad 6 smd rect (at 0.9 -0.75 270) (size 0.6 0.6) (layers F.Cu F.Paste F.Mask)
-      (net 16 "Net-(C9-Pad1)"))
-    (pad 2 smd rect (at -0.9 0 270) (size 0.6 0.4) (layers F.Cu F.Paste F.Mask))
-    (pad 5 smd rect (at 0.9 0 270) (size 0.6 0.4) (layers F.Cu F.Paste F.Mask))
-  )
   (module CRYSTAL_3225_4 (layer F.Cu)
     (at 132.6 86.3)
@@
     )
   )
-  (module SOT23-6 (layer F.Cu)
-    (at 140.2 84.1 90)
-    (fp_text reference U2 (at -1.69926 -1.30048 180) (layer F.Fab)
-      (effects (font (size 0.29972 0.29972) (thickness 0.07493)))
-    )
-    (fp_text value MCP3425 (at 0 -0.3 90) (layer F.Fab)
-      (effects (font (size 0.29972 0.29972) (thickness 0.07493)))
-    )
-    (fp_line (start -1.5494 0.20066) (end -0.52578 0.20066) (layer F.Fab) (width 0.09906))
-    (fp_line (start -0.52578 0.20066) (end -0.52578 0.8509) (layer F.Fab) (width 0.09906))
-    (fp_line (start -1.5494 -0.8509) (end 1.5494 -0.8509) (layer F.Fab) (width 0.09906))
-    (fp_line (start 1.5494 -0.8509) (end 1.5494 0.8509) (layer F.Fab) (width 0.09906))
-    (fp_line (start 1.5494 0.8509) (end -1.5494 0.8509) (layer F.Fab) (width 0.09906))
-    (fp_line (start -1.5494 0.8509) (end -1.5494 -0.8509) (layer F.Fab) (width 0.09906))
-    (pad 1 smd rect (at -0.94996 1.19888 90) (size 0.50038 0.8001) (layers F.Cu F.Paste F.Mask)
-      (net 6 "Net-(R3-Pad1)") (clearance 0.14986))
-    (pad 2 smd rect (at 0 1.19888 90) (size 0.50038 0.8001) (layers F.Cu F.Paste F.Mask)
-      (net 1 GND) (clearance 0.14986))
-    (pad 3 smd rect (at 0.94996 1.19888 90) (size 0.50038 0.8001) (layers F.Cu F.Paste F.Mask)
-      (net 12 SCL) (clearance 0.14986))
-    (pad 6 smd rect (at -0.94996 -1.19888 90) (size 0.50038 0.8001) (layers F.Cu F.Paste F.Mask)
-      (net 23 "Net-(R6-Pad1)") (clearance 0.14986))
-    (pad 4 smd rect (at 0.94996 -1.19888 90) (size 0.50038 0.8001) (layers F.Cu F.Paste F.Mask)
-      (net 13 SDA) (clearance 0.14986))
-    (pad 5 smd rect (at 0 -1.19888 90) (size 0.50038 0.8001) (layers F.Cu F.Paste F.Mask)
-      (net 15 "Net-(C6-Pad1)") (clearance 0.14986))
-  )
   (module kicad-libraries:Logo_31x31 (layer B.Cu)
     (at 137.6 88.15 180)
@@
       (xy 2.3114 -1.41732) (xy 2.3114 -1.67132) (xy 2.3114 -1.67132)) (layer B.SilkS) (width 0.00254))
   )
+  (module kicad-libraries:SOT23-6 (layer F.Cu)
+    (at 140.2 84.1 90)
+    (fp_text reference U2 (at -1.69926 -1.30048 180) (layer F.Fab)
+      (effects (font (size 0.29972 0.29972) (thickness 0.07493)))
+    )
+    (fp_text value MCP3425 (at 0 -0.3 90) (layer F.Fab)
+      (effects (font (size 0.29972 0.29972) (thickness 0.07493)))
+    )
+    (fp_line (start -1.5494 0.20066) (end -0.52578 0.20066) (layer F.Fab) (width 0.09906))
+    (fp_line (start -0.52578 0.20066) (end -0.52578 0.8509) (layer F.Fab) (width 0.09906))
+    (fp_line (start -1.5494 -0.8509) (end 1.5494 -0.8509) (layer F.Fab) (width 0.09906))
+    (fp_line (start 1.5494 -0.8509) (end 1.5494 0.8509) (layer F.Fab) (width 0.09906))
+    (fp_line (start 1.5494 0.8509) (end -1.5494 0.8509) (layer F.Fab) (width 0.09906))
+    (fp_line (start -1.5494 0.8509) (end -1.5494 -0.8509) (layer F.Fab) (width 0.09906))
+    (pad 1 smd rect (at -0.94996 1.19888 90) (size 0.50038 0.8001) (layers F.Cu F.Paste F.Mask)
+      (net 6 "Net-(R3-Pad1)") (clearance 0.14986))
+    (pad 2 smd rect (at 0 1.19888 90) (size 0.50038 0.8001) (layers F.Cu F.Paste F.Mask)
+      (net 1 GND) (clearance 0.14986))
+    (pad 3 smd rect (at 0.94996 1.19888 90) (size 0.50038 0.8001) (layers F.Cu F.Paste F.Mask)
+      (net 12 SCL) (clearance 0.14986))
+    (pad 6 smd rect (at -0.94996 -1.19888 90) (size 0.50038 0.8001) (layers F.Cu F.Paste F.Mask)
+      (net 23 "Net-(R6-Pad1)") (clearance 0.14986))
+    (pad 4 smd rect (at 0.94996 -1.19888 90) (size 0.50038 0.8001) (layers F.Cu F.Paste F.Mask)
+      (net 13 SDA) (clearance 0.14986))
+    (pad 5 smd rect (at 0 -1.19888 90) (size 0.50038 0.8001) (layers F.Cu F.Paste F.Mask)
+      (net 15 "Net-(C6-Pad1)") (clearance 0.14986))
+    (model Housing_SOT_SOD/SOT-23-6.wrl
+      (at (xyz 0 0 0))
+      (scale (xyz 1 1 1))
+      (rotate (xyz 90 180 90))
+    )
+  )
+  (module kicad-libraries:SOT363 (layer F.Cu)
+    (at 136.7 91 270)
+    (attr smd)
+    (fp_text reference D2 (at 0.35 0 360) (layer F.Fab)
+      (effects (font (size 0.2 0.2) (thickness 0.05)))
+    )
+    (fp_text value BAT54TW (at 0.025 0.125 360) (layer F.Fab)
+      (effects (font (size 0.2 0.2) (thickness 0.05)))
+    )
+    (fp_circle (center -0.25 -0.7) (end -0.2 -0.65) (layer F.Fab) (width 0.05))
+    (fp_line (start -0.65 -1.1) (end 0.65 -1.1) (layer F.Fab) (width 0.05))
+    (fp_line (start 0.65 -1.1) (end 0.65 1.1) (layer F.Fab) (width 0.05))
+    (fp_line (start 0.65 1.1) (end -0.65 1.1) (layer F.Fab) (width 0.05))
+    (fp_line (start -0.65 1.1) (end -0.65 -1.1) (layer F.Fab) (width 0.05))
+    (pad 1 smd rect (at -0.9 -0.75 270) (size 0.6 0.6) (layers F.Cu F.Paste F.Mask)
+      (net 19 "Net-(D2-Pad1)"))
+    (pad 3 smd rect (at -0.9 0.75 270) (size 0.6 0.6) (layers F.Cu F.Paste F.Mask)
+      (net 25 SIG))
+    (pad 4 smd rect (at 0.9 0.75 270) (size 0.6 0.6) (layers F.Cu F.Paste F.Mask)
+      (net 17 "Net-(C10-Pad1)"))
+    (pad 6 smd rect (at 0.9 -0.75 270) (size 0.6 0.6) (layers F.Cu F.Paste F.Mask)
+      (net 16 "Net-(C9-Pad1)"))
+    (pad 2 smd rect (at -0.9 0 270) (size 0.6 0.4) (layers F.Cu F.Paste F.Mask))
+    (pad 5 smd rect (at 0.9 0 270) (size 0.6 0.4) (layers F.Cu F.Paste F.Mask))
+    (model Housing_SOT_SOD/SOT-363.wrl
+      (at (xyz 0 0 -0.002))
+      (scale (xyz 1 1 1))
+      (rotate (xyz 90 180 90))
+    )
+  )
   (gr_line (start 131 147.35) (end 136 152.35) (angle 90) (layer F.SilkS) (width 0.2))

Commit message: change footprints
Parts:
- C2: footprint C0402E -> kicad-libraries:C0402F
Other:
- outline, holes or cut-outs redrawn
Changed lines of the file:
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@@
-(kicad_pcb (version 4) (host pcbnew 4.0.2+dfsg1-stable)
+(kicad_pcb (version 4) (host pcbnew 4.0.7-e2-6376~58~ubuntu17.04.1)
   (general
     (links 71)
     (no_connects 0)
-    (area 128.424999 67.274999 143.575001 152.425001)
+    (area 128.349159 66.35 394.84286 254.69)
     (thickness 1.6)
-    (drawings 63)
+    (drawings 59)
     (tracks 247)
     (zones 0)
@@
   )
   (layers
-    (0 F.Cu signal hide)
+    (0 F.Cu signal)
     (31 B.Cu signal hide)
     (32 B.Adhes user)
@@
     )
   )
-  (module C0402E (layer F.Cu)
-    (at 132.4 74.25 90)
-    (attr smd)
-    (fp_text reference C2 (at 0 0.125 90) (layer F.Fab)
-      (effects (font (size 0.2 0.2) (thickness 0.05)))
-    )
-    (fp_text value TBD (at 0 -0.275 90) (layer F.Fab)
-      (effects (font (size 0.2 0.2) (thickness 0.05)))
-    )
-    (fp_line (start -0.8509 -0.44958) (end 0.8509 -0.44958) (layer F.Fab) (width 0.001))
-    (fp_line (start 0.8509 -0.44958) (end 0.8509 0.44958) (layer F.Fab) (width 0.001))
-    (fp_line (start 0.8509 0.44958) (end -0.8509 0.44958) (layer F.Fab) (width 0.001))
-    (fp_line (start -0.8509 0.44958) (end -0.8509 -0.44958) (layer F.Fab) (width 0.001))
-    (pad 1 smd rect (at -0.65 0 90) (size 0.7 0.9) (layers F.Cu F.Paste F.Mask)
-      (net 1 GND))
-    (pad 2 smd rect (at 0.65 0 90) (size 0.7 0.9) (layers F.Cu F.Paste F.Mask)
-      (net 14 "Net-(C2-Pad2)"))
-    (model Capacitors_SMD/C_0402.wrl
-      (at (xyz 0 0 0))
-      (scale (xyz 1 1 1))
-      (rotate (xyz 0 0 0))
-    )
-  )
   (module C0603F (layer F.Cu)
     (at 138.6 75.9 180)
@@
     )
   )
+  (module kicad-libraries:C0402F (layer F.Cu)
+    (at 132.4 74.25 90)
+    (fp_text reference C2 (at 0.1 0.15 90) (layer F.Fab)
+      (effects (font (size 0.2 0.2) (thickness 0.05)))
+    )
+    (fp_text value TBD (at 0 -0.15 90) (layer F.Fab)
+      (effects (font (size 0.2 0.2) (thickness 0.05)))
+    )
+    (fp_line (start -0.9 -0.45) (end 0.9 -0.45) (layer F.Fab) (width 0.025))
+    (fp_line (start 0.9 -0.45) (end 0.9 0.45) (layer F.Fab) (width 0.025))
+    (fp_line (start 0.9 0.45) (end -0.9 0.45) (layer F.Fab) (width 0.025))
+    (fp_line (start -0.9 0.45) (end -0.9 -0.45) (layer F.Fab) (width 0.025))
+    (pad 2 smd rect (at 0.5 0 90) (size 0.6 0.7) (layers F.Cu F.Paste F.Mask)
+      (net 14 "Net-(C2-Pad2)"))
+    (pad 1 smd rect (at -0.5 0 90) (size 0.6 0.7) (layers F.Cu F.Paste F.Mask)
+      (net 1 GND))
+  )
+  (gr_line (start 131 93.85) (end 131 147.35) (angle 90) (layer Edge.Cuts) (width 0.15))
+  (gr_line (start 141 147.35) (end 141 93.85) (angle 90) (layer Edge.Cuts) (width 0.15))
+  (gr_line (start 128.5 91.35) (end 131 93.85) (angle 90) (layer Edge.Cuts) (width 0.15))
+  (gr_line (start 143.5 91.35) (end 141 93.85) (angle 90) (layer Edge.Cuts) (width 0.15))
   (gr_line (start 131 147.35) (end 136 152.35) (angle 90) (layer F.SilkS) (width 0.2))
   (gr_text 0 (at 136 146.35) (layer B.SilkS)
@@
   (gr_line (start 141 142.35) (end 131 142.35) (angle 90) (layer F.SilkS) (width 0.2))
   (gr_line (start 141 147.35) (end 131 147.35) (angle 90) (layer F.SilkS) (width 0.2))
-  (gr_line (start 131 147.35) (end 131 93.35) (angle 90) (layer Edge.Cuts) (width 0.15))
-  (gr_line (start 141 93.35) (end 141 147.35) (angle 90) (layer Edge.Cuts) (width 0.15))
   (gr_line (start 143.5 68.35) (end 143.5 91.35) (angle 90) (layer Edge.Cuts) (width 0.15))
   (gr_line (start 129.5 67.35) (end 142.5 67.35) (angle 90) (layer Edge.Cuts) (width 0.15))
   (gr_line (start 128.5 91.35) (end 128.5 68.35) (angle 90) (layer Edge.Cuts) (width 0.15))
-  (gr_line (start 129.5 92.35) (end 130 92.35) (angle 90) (layer Edge.Cuts) (width 0.15))
-  (gr_line (start 142 92.35) (end 142.5 92.35) (angle 90) (layer Edge.Cuts) (width 0.15))
   (gr_arc (start 142.5 68.35) (end 142.5 67.35) (angle 90) (layer Edge.Cuts) (width 0.15))
   (gr_arc (start 129.5 68.35) (end 128.5 68.35) (angle 90) (layer Edge.Cuts) (width 0.15))
-  (gr_arc (start 129.5 91.35) (end 129.5 92.35) (angle 90) (layer Edge.Cuts) (width 0.15))
-  (gr_arc (start 142.5 91.35) (end 143.5 91.35) (angle 90) (layer Edge.Cuts) (width 0.15))
-  (gr_arc (start 130 93.35) (end 130 92.35) (angle 90) (layer Edge.Cuts) (width 0.15))
-  (gr_arc (start 142 93.35) (end 141 93.35) (angle 90) (layer Edge.Cuts) (width 0.15))
   (gr_line (start 136 152.35) (end 141 147.35) (angle 90) (layer Edge.Cuts) (width 0.15))
   (gr_line (start 136 152.35) (end 131 147.35) (angle 90) (layer Edge.Cuts) (width 0.15))
@@
   (via (at 140.325 76.975) (size 0.7) (drill 0.25) (layers F.Cu B.Cu) (net 1))
   (segment (start 140.15 77.15) (end 140.325 76.975) (width 0.254) (layer F.Cu) (net 1))
-  (segment (start 132.4 74.9) (end 132.4 75.325) (width 0.254) (layer F.Cu) (net 1))
-  (via (at 132.15 75.6) (size 0.7) (drill 0.25) (layers F.Cu B.Cu) (net 1))
-  (segment (start 132.15 75.575) (end 132.15 75.6) (width 0.254) (layer F.Cu) (net 1))
-  (segment (start 132.4 75.325) (end 132.15 75.575) (width 0.254) (layer F.Cu) (net 1))
   (segment (start 135.15 78.35) (end 135.15 79.65) (width 0.254) (layer F.Cu) (net 1))
   (segment (start 133.85 78.35) (end 135.15 78.35) (width 0.254) (layer F.Cu) (net 1))
@@
   (segment (start 133.1 90.35) (end 132.3 90.35) (width 0.5) (layer F.Cu) (net 1))
   (via (at 132.3 90.35) (size 0.7) (drill 0.25) (layers F.Cu B.Cu) (net 1))
+  (segment (start 132.4 74.9) (end 132.4 75.325) (width 0.254) (layer F.Cu) (net 1))
+  (via (at 132.15 75.6) (size 0.7) (drill 0.25) (layers F.Cu B.Cu) (net 1))
+  (segment (start 132.15 75.575) (end 132.15 75.6) (width 0.254) (layer F.Cu) (net 1))
+  (segment (start 132.4 75.325) (end 132.15 75.575) (width 0.254) (layer F.Cu) (net 1))
   (segment (start 131.05 84.1) (end 131.425 84.1) (width 0.254) (layer F.Cu) (net 2))
   (segment (start 131.425 84.1) (end 131.7 84.375) (width 0.254) (layer F.Cu) (net 2))
@@
   (segment (start 138.34996 83.15004) (end 139.00112 83.15004) (width 0.254) (layer F.Cu) (net 13))
   (segment (start 138.19888 83.30112) (end 138.34996 83.15004) (width 0.254) (layer F.Cu) (net 13))
-  (segment (start 132.25 71.7) (end 132.25 72.95) (width 0.254) (layer F.Cu) (net 14))
   (segment (start 132.4 73.1) (end 132.4 73.6) (width 0.254) (layer F.Cu) (net 14))
+  (segment (start 132.9 73.6) (end 132.4 73.6) (width 0.254) (layer F.Cu) (net 14))
+  (segment (start 132.25 71.7) (end 132.25 72.95) (width 0.254) (layer F.Cu) (net 14))
   (segment (start 132.25 72.95) (end 132.4 73.1) (width 0.254) (layer F.Cu) (net 14))
   (segment (start 133.4507 73.825) (end 133.125 73.825) (width 0.254) (layer F.Cu) (net 14))
-  (segment (start 132.9 73.6) (end 132.4 73.6) (width 0.254) (layer F.Cu) (net 14))
   (segment (start 133.125 73.825) (end 132.9 73.6) (width 0.254) (layer F.Cu) (net 14))
   (segment (start 138.65 80.4) (end 138.75 80.4) (width 0.254) (layer F.Cu) (net 15))
